Commit message: Added flange deg 90 for the mia hand

File: fr3_miahand_description/robots/common/franka_robot.xacro (robot description, xacro)
@@ -1,47 +1,78 @@
 <?xml version='1.0' encoding='utf-8'?>
 <robot xmlns:xacro="http://www.ros.org/wiki/xacro">
-  <xacro:macro name="franka_robot" params="arm_id joint_limits parent:='world' xyz:='0 0 0' rpy:='0 0 0' gazebo:=false">
+  <xacro:macro name="franka_robot"
+    params="arm_id joint_limits parent:='world' xyz:='0 0 0' rpy:='0 0 0' gazebo:=false">
     <xacro:include filename="$(find fr3_miahand_description)/robots/common/utils.xacro" />
     <xacro:include filename="$(find fr3_miahand_description)/robots/common/franka_arm.xacro" />
-    <xacro:franka_arm arm_id="${arm_id}" safety_distance="0.03" gazebo="${gazebo}" joint_limits="${joint_limits}"/>
+    <xacro:franka_arm arm_id="${arm_id}" safety_distance="0.03" gazebo="${gazebo}"
+      joint_limits="${joint_limits}" />
+    <xacro:if value="${parent != ''}">
+      <!-- Gazebo requires a joint to a link called "world" for statically mounted robots -->
+      <xacro:if value="${parent == 'world'}">
+        <link name="${parent}" />
+      </xacro:if>
+      <xacro:table parent="$(arg parent)">
+        <origin xyz="0.0 0.0 0.6" rpy="0.0 0.0 0.0" />
+      </xacro:table>
+      <!-- <joint name="${parent}_joint" type="fixed">
+          <origin xyz="${xyz}" rpy="${rpy}" />
+          <parent link="${parent}" />
+          <child link="${arm_id}_link0" />
+        </joint> -->
+      <joint name="j_base_link_table" type="fixed">
+        <origin xyz="${xyz}" rpy="${rpy}" />
+        <parent link="base_link_table" />
+        <child link="${arm_id}_link0" />
+      </joint>
+    </xacro:if>
     <!-- Define additional Gazebo tags -->
     <xacro:if value="${gazebo}">
-      <xacro:if value="${parent != ''}">
-        <!-- Gazebo requires a joint to a link called "world" for statically mounted robots -->
-        <xacro:if value="${parent == 'world'}">
-          <link name="${parent}" />
-        </xacro:if>
-        <joint name="${parent}_joint" type="fixed">
-          <origin xyz="${xyz}" rpy="${rpy}" />
-          <parent link="${parent}" />
-          <child  link="${arm_id}_link0" />
-        </joint>
-      </xacro:if>
-      <xacro:gazebo-joint joint="${arm_id}_joint1" transmission="hardware_interface/PositionJointInterface" />
-      <xacro:gazebo-joint joint="${arm_id}_joint2" transmission="hardware_interface/PositionJointInterface" />
-      <xacro:gazebo-joint joint="${arm_id}_joint3" transmission="hardware_interface/PositionJointInterface" />
-      <xacro:gazebo-joint joint="${arm_id}_joint4" transmission="hardware_interface/PositionJointInterface" />
-      <xacro:gazebo-joint joint="${arm_id}_joint5" transmission="hardware_interface/PositionJointInterface" />
-      <xacro:gazebo-joint joint="${arm_id}_joint6" transmission="hardware_interface/PositionJointInterface" />
-      <xacro:gazebo-joint joint="${arm_id}_joint7" transmission="hardware_interface/PositionJointInterface" />
-      <xacro:gazebo-joint joint="${arm_id}_joint1" transmission="hardware_interface/VelocityJointInterface" />
-      <xacro:gazebo-joint joint="${arm_id}_joint2" transmission="hardware_interface/VelocityJointInterface" />
-      <xacro:gazebo-joint joint="${arm_id}_joint3" transmission="hardware_interface/VelocityJointInterface" />
-      <xacro:gazebo-joint joint="${arm_id}_joint4" transmission="hardware_interface/VelocityJointInterface" />
-      <xacro:gazebo-joint joint="${arm_id}_joint5" transmission="hardware_interface/VelocityJointInterface" />
-      <xacro:gazebo-joint joint="${arm_id}_joint6" transmission="hardware_interface/VelocityJointInterface" />
-      <xacro:gazebo-joint joint="${arm_id}_joint7" transmission="hardware_interface/VelocityJointInterface" />
-      <xacro:gazebo-joint joint="${arm_id}_joint1" transmission="hardware_interface/EffortJointInterface" />
-      <xacro:gazebo-joint joint="${arm_id}_joint2" transmission="hardware_interface/EffortJointInterface" />
-      <xacro:gazebo-joint joint="${arm_id}_joint3" transmission="hardware_interface/EffortJointInterface" />
-      <xacro:gazebo-joint joint="${arm_id}_joint4" transmission="hardware_interface/EffortJointInterface" />
-      <xacro:gazebo-joint joint="${arm_id}_joint5" transmission="hardware_interface/EffortJointInterface" />
-      <xacro:gazebo-joint joint="${arm_id}_joint6" transmission="hardware_interface/EffortJointInterface" />
-      <xacro:gazebo-joint joint="${arm_id}_joint7" transmission="hardware_interface/EffortJointInterface" />
+      <xacro:gazebo-joint joint="${arm_id}_joint1"
+        transmission="hardware_interface/PositionJointInterface" />
+      <xacro:gazebo-joint joint="${arm_id}_joint2"
+        transmission="hardware_interface/PositionJointInterface" />
+      <xacro:gazebo-joint joint="${arm_id}_joint3"
+        transmission="hardware_interface/PositionJointInterface" />
+      <xacro:gazebo-joint joint="${arm_id}_joint4"
+        transmission="hardware_interface/PositionJointInterface" />
+      <xacro:gazebo-joint joint="${arm_id}_joint5"
+        transmission="hardware_interface/PositionJointInterface" />
+      <xacro:gazebo-joint joint="${arm_id}_joint6"
+        transmission="hardware_interface/PositionJointInterface" />
+      <xacro:gazebo-joint joint="${arm_id}_joint7"
+        transmission="hardware_interface/PositionJointInterface" />
+      <xacro:gazebo-joint joint="${arm_id}_joint1"
+        transmission="hardware_interface/VelocityJointInterface" />
+      <xacro:gazebo-joint joint="${arm_id}_joint2"
+        transmission="hardware_interface/VelocityJointInterface" />
+      <xacro:gazebo-joint joint="${arm_id}_joint3"
+        transmission="hardware_interface/VelocityJointInterface" />
+      <xacro:gazebo-joint joint="${arm_id}_joint4"
+        transmission="hardware_interface/VelocityJointInterface" />
+      <xacro:gazebo-joint joint="${arm_id}_joint5"
+        transmission="hardware_interface/VelocityJointInterface" />
+      <xacro:gazebo-joint joint="${arm_id}_joint6"
+        transmission="hardware_interface/VelocityJointInterface" />
+      <xacro:gazebo-joint joint="${arm_id}_joint7"
+        transmission="hardware_interface/VelocityJointInterface" />
+      <xacro:gazebo-joint joint="${arm_id}_joint1"
+        transmission="hardware_interface/EffortJointInterface" />
+      <xacro:gazebo-joint joint="${arm_id}_joint2"
+        transmission="hardware_interface/EffortJointInterface" />
+      <xacro:gazebo-joint joint="${arm_id}_joint3"
+        transmission="hardware_interface/EffortJointInterface" />
+      <xacro:gazebo-joint joint="${arm_id}_joint4"
+        transmission="hardware_interface/EffortJointInterface" />
+      <xacro:gazebo-joint joint="${arm_id}_joint5"
+        transmission="hardware_interface/EffortJointInterface" />
+      <xacro:gazebo-joint joint="${arm_id}_joint6"
+        transmission="hardware_interface/EffortJointInterface" />
+      <xacro:gazebo-joint joint="${arm_id}_joint7"
+        transmission="hardware_interface/EffortJointInterface" />
       <xacro:transmission-franka-state arm_id="${arm_id}" />
       <xacro:transmission-franka-model arm_id="${arm_id}"
-         root="${arm_id}_joint1"
-         tip="${arm_id}_joint8"
-       />
+        root="${arm_id}_joint1"
+        tip="${arm_id}_joint8"
+      />
       <gazebo>
         <plugin name="gazebo_ros_control" filename="libgazebo_ros_control.so">

File: fr3_miahand_description/robots/common/properties.xacro (robot description, xacro)
@@ -1,4 +1,4 @@
 <?xml version="1.0"?>
-<robot name="macroed" xmlns:xacro="http://ros.org/wiki/xacro">
+<robot name="utils" xmlns:xacro="http://ros.org/wiki/xacro">
     <xacro:property name="pi" value="3.1415" />
 </robot>

File: fr3_miahand_description/robots/common/utils.xacro (robot description, xacro)
@@ -38,10 +38,10 @@
       <visual>
         <geometry>
-          <mesh filename="package://${description_pkg}/meshes/visual/${name}.dae" />
+          <mesh filename="package://${description_pkg}/meshes/fr3/visual/${name}.dae" />
         </geometry>
       </visual>
       <collision>
         <geometry>
-          <mesh filename="package://${description_pkg}/meshes/collision/${name}.stl" />
+          <mesh filename="package://${description_pkg}/meshes/fr3/collision/${name}.stl" />
         </geometry>
       </collision>

File: fr3_miahand_description/robots/fr3/fr3_miahand.urdf.xacro (robot description, xacro)
@@ -2,25 +2,47 @@
 <robot xmlns:xacro="http://www.ros.org/wiki/xacro" name="fr3">
   <xacro:include filename="$(find fr3_miahand_description)/robots/common/properties.xacro" />
+  <!-- Include macro table -->
+  <xacro:include filename="$(find fr3_miahand_description)/robots/extra/table.xacro" />
   <xacro:include filename="$(find fr3_miahand_description)/robots/common/franka_robot.xacro" />
   <xacro:include filename="$(find fr3_miahand_description)/robots/mia/mia_hand_flange.xacro" />
+  <!-- Include macro for flange deg 90 -->
+  <xacro:include filename="$(find fr3_miahand_description)/robots/common/flange_deg_90.xacro" />
   <!-- Name for this robot -->
   <xacro:arg name="arm_id" default="fr3" />
   <!-- Is the robot being simulated in gazebo?" -->
   <xacro:arg name="gazebo" default="false" />
-  <!-- If `gazebo` arg is set, to which frame shall $(arm_id)_link0 be parented. Empty string for not fixing at all -->
+  <!-- If `gazebo` arg is set, to which frame shall $(arm_id)_link0 be parented. Empty string for
+  not fixing at all -->
   <xacro:arg name="parent" default="world" />
-  <!-- If `gazebo` arg is set and `parent` not empty, what position offset between `parent` & $(arm_id)_link0 -->
-  <xacro:arg name="xyz" default="0 0 0" />
-  <!-- If `gazebo` arg is set and `parent` not empty, what rotation offset between `parent` & $(arm_id)_link0 -->
+  <!-- If `gazebo` arg is set and `parent` not empty, what position offset between `parent` &
+  base_link_table -->
+  <xacro:arg name="xyz" default="0 0 0.024" />
+  <!-- If `gazebo` arg is set and `parent` not empty, what rotation offset between `parent` &
+  $(arm_id)_link0 -->
   <xacro:arg name="rpy" default="0 0 0" />
+  <xacro:arg name="flange_deg_90" default="false" />
   <!-- fr3 macro -->
   <xacro:franka_robot arm_id="$(arg arm_id)"
-                      joint_limits="${xacro.load_yaml('$(find fr3_miahand_description)/robots/fr3/joint_limits.yaml')}"
-                      gazebo="$(arg gazebo)"
-                      parent="$(arg parent)"
-                      xyz="$(arg xyz)"
-                      rpy="$(arg rpy)">
+    joint_limits="${xacro.load_yaml('$(find fr3_miahand_description)/robots/fr3/joint_limits.yaml')}"
+    gazebo="$(arg gazebo)"
+    parent="$(arg parent)"
+    xyz="$(arg xyz)"
+    rpy="$(arg rpy)">
   </xacro:franka_robot>
-  <!-- mia hand macro with URFlange -->
-  <xacro:mia_hand_flange parent="fr3_link8" gazebo="$(arg gazebo)" />
+  <!-- mia hand macro with URFlange  -->
+  <!-- Check if you want to add also the 90 deg flange -->
+  <xacro:if value="$(arg flange_deg_90)">
+    <!-- Add the 90 degree flange between fr3_link8 and the mia hand -->
+    <xacro:flange_deg_90 parent="fr3_link8" />
+    <!-- Add mia hand -->
+    <xacro:mia_hand_flange parent="attach_link" gazebo="$(arg gazebo)">
+      <origin xyz="0.0 0.0 0.0" rpy="${pi / 2.0} ${-pi / 2.0} 0.0" />
+    </xacro:mia_hand_flange>
+  </xacro:if>
+  <xacro:unless value="$(arg flange_deg_90)">
+    <!-- Add mia hand -->
+    <xacro:mia_hand_flange parent="fr3_link8" gazebo="$(arg gazebo)">
+      <origin xyz="0.0 0.0 0.0" rpy="0.0 0.0 ${pi}" />
+    </xacro:mia_hand_flange>
+  </xacro:unless>
 </robot>

File: fr3_miahand_description/robots/mia/mia_hand_flange.xacro (robot description, xacro)
@@ -1,5 +1,5 @@
 <?xml version='1.0' encoding='utf-8'?>
 <robot xmlns:xacro="http://www.ros.org/wiki/xacro">
-    <xacro:macro name="mia_hand_flange" params="parent gazebo">
+    <xacro:macro name="mia_hand_flange" params="parent gazebo *origin">
         <!-- true it loads robot model with default config provided by default yaml file
     False it loads calibrated robot model configuaration yaml file.
@@ -49,5 +49,5 @@
         </link>
         <joint name="j_fr3_link8_to_URflange" type="fixed">
-            <origin xyz="0.0 0.0 0.0" rpy="0.0 0.0 ${pi}" />
+            <xacro:insert_block name="origin"/>
             <parent link="${parent}" />
             <child link="URflange" />

Commit message: Modified rsp to take into account the remapping of the mia hand joint states(index thumb).

File: fr3_miahand_description/robots/common/franka_robot.xacro (robot description, xacro)
@@ -13,5 +13,5 @@
       </xacro:if>
       <xacro:table parent="$(arg parent)">
-        <origin xyz="0.0 0.0 0.6" rpy="0.0 0.0 0.0" />
+        <origin xyz="0.0 0.0 ${heigth_leg_table}" rpy="0.0 0.0 0.0" />
       </xacro:table>
       <!-- <joint name="${parent}_joint" type="fixed">

File: fr3_miahand_description/robots/common/properties.xacro (robot description, xacro)
@@ -2,3 +2,6 @@
 <robot name="utils" xmlns:xacro="http://ros.org/wiki/xacro">
     <xacro:property name="pi" value="3.1415" />
+    <xacro:property name="heigth_robot_table" value="0.024" />
+    <xacro:property name="heigth_leg_table" value="0.6" />
+    <xacro:property name="base_link_table_x" value="0.5" />
 </robot>

File: fr3_miahand_description/robots/fr3/fr3_miahand.urdf.xacro (robot description, xacro)
@@ -17,7 +17,7 @@
   <!-- If `gazebo` arg is set and `parent` not empty, what position offset between `parent` &
   base_link_table -->
-  <xacro:arg name="xyz" default="0 0 0.024" />
+  <xacro:arg name="xyz" default="${-base_link_table_x} 0 ${heigth_robot_table}" />
   <!-- If `gazebo` arg is set and `parent` not empty, what rotation offset between `parent` &
-  $(arm_id)_link0 -->
+  base_link_table -->
   <xacro:arg name="rpy" default="0 0 0" />
   <xacro:arg name="flange_deg_90" default="false" />
